File: src/printed-circuit-boards/FLWSB-connector-board/FLWSB-connector-board.kicad_pcb (KiCad board)
At the start: 2 copper layers, 43 parts, among them IC1 LDL1117S33R, J1 Conn_01x04_Male, J2 Conn_01x03_Male, J3 SDS011_JST-XH-5, J4 Conn_01x03_Male, J5 Conn_01x04_Male, J6 Conn_01x03_Male, U1 FLWSB-SAMDaaNo21-v1

Commit message: Update connector board v1.1
Parts:
- removed J6: Conn_01x03_Male, Connector_PinHeader_2.54mm:PinHeader_1x03_P2.54mm_Vertical
- added B5: GY-SGP41_Breakout, Connector_PinHeader_2.54mm:PinHeader_1x04_P2.54mm_Vertical, F.Cu at (196.3, 355.0)
- added B6: SCD41_Breakout, Connector_PinHeader_2.54mm:PinHeader_1x04_P2.54mm_Vertical, F.Cu at (201.0, 355.0)
- added B7: DHT22_Breakout, Connector_PinHeader_2.54mm:PinHeader_1x04_P2.54mm_Vertical, F.Cu at (205.6, 355.0)
- added C10: 100nF, Capacitor_SMD:C_0805_2012Metric_Pad1.18x1.45mm_HandSolder, F.Cu at (210.4, 357.1)
- added C9: 100nF, Capacitor_SMD:C_0805_2012Metric_Pad1.18x1.45mm_HandSolder, F.Cu at (210.4, 354.1)
- B2: value CCS811_Breakout -> GY-NEO6MV2_Breakout; footprint Component_Library_Bavo:CCS811_Breakout -> Connector_PinHeader_2.54mm:PinHeader_1x04_P2.54mm_Vertical
- B3: value BME280_Breakout -> CCS811_Breakout; footprint Component_Library_Bavo:BM280_Breakout -> Component_Library_Bavo:CCS811_Breakout
- B4: value DHT22_Breakout -> BME280_Breakout; footprint Connector_PinHeader_2.54mm:PinHeader_1x04_P2.54mm_Vertical -> Component_Library_Bavo:BM280_Breakout
- C4: value 100nF -> 1µF
- J1, J5: value Conn_01x04_Male -> Conn_01x03_Male; footprint Connector_PinHeader_2.54mm:PinHeader_1x04_P2.54mm_Vertical -> Connector_PinHeader_2.54mm:PinHeader_1x03_P2.54mm_Vertical
- J2: value Conn_01x03_Male -> SDS011_JST-XH-5; footprint Connector_PinHeader_2.54mm:PinHeader_1x03_P2.54mm_Vertical -> Connector_JST:JST_XH_B5B-XH-A_1x05_P2.50mm_Vertical
- J3: value SDS011_JST-XH-5 -> Conn_01x03_Male; footprint Connector_JST:JST_XH_B5B-XH-A_1x05_P2.50mm_Vertical -> Connector_PinHeader_2.54mm:PinHeader_1x03_P2.54mm_Vertical
- J4: value Conn_01x03_Male -> SPS30_JST-ZHR-5; footprint Connector_PinHeader_2.54mm:PinHeader_1x03_P2.54mm_Vertical -> Connector_JST:JST_XH_B5B-XH-A_1x05_P2.50mm_Vertical
Connections:
- B2 pad 2: GND2 -> S5TX-EXTRA_RX
- B2 pad 3: SCL -> S5RX-EXTRA_TX
- B2 pad 4: SDA -> GND2
- B4 pad 2: DATA -> GND2
- B4 pad 3: unconnected-(B4-Pad3) -> SCL
- B4 pad 4: GND2 -> SDA
- C4 pad 1: +3V3 -> +5V
- J1 pad 1: S5RX -> S2TX-LoRa_RX
- J1 pad 2: S5TX -> S2RX-LoRa_TX
- J1 pad 3: GND2 -> RST-LoRa
- J2 pad 1: S2RX-LoRa -> S0RX-SDS_TX
- J2 pad 2: S2TX-LoRa -> SOTX-SDS_RX
- J2 pad 3: RST-LoRa -> GND2
- J3 pad 1: S0TX-SDS -> +5V
- J3 pad 2: S0RX-SDS -> +3V3
- J4 pad 2: +3V3 -> SDA
- J4 pad 3: GND2 -> SCL
- J5 pad 1: SDA -> Net-(J5-Pad1)
- J5 pad 2: SCL -> Net-(J5-Pad2)
- J5 pad 3: GND2 -> GND1
- R10 pad 1: Net-(U1-Pad29) -> Net-(J5-Pad2)
- R3 pad 2: S5TX -> S5RX-EXTRA_TX
- R4 pad 2: S5RX -> S5TX-EXTRA_RX
- R5 pad 2: S2TX-LoRa -> S2RX-LoRa_TX
- R6 pad 2: S2RX-LoRa -> S2TX-LoRa_RX
- R9 pad 1: Net-(U1-Pad30) -> Net-(J5-Pad1)
- U1 pad 10: S2TX-LoRa -> S2TX-LoRa_RX
- U1 pad 11: S2RX-LoRa -> S2RX-LoRa_TX
- U1 pad 24: S5TX -> S5RX-EXTRA_TX
- U1 pad 25: S5RX -> S5TX-EXTRA_RX
- U1 pad 29: Net-(U1-Pad29) -> Net-(J5-Pad2)
- U1 pad 30: Net-(U1-Pad30) -> Net-(J5-Pad1)
- U1 pad 6: S0TX-SDS -> SOTX-SDS_RX
- U1 pad 7: SORX-SDS -> S0RX-SDS_TX
