File: src/printed-circuit-boards/FLWSB-connector-board/FLWSB-connector-board.kicad_sch (KiCad schematic)
At the start: 43 parts

Commit message: Update connector board v1.1
Parts:
- removed J1, J5: (no value), symbol Connector:Conn_01x04_Male
- added B2: GY-NEO6MV2_Breakout, Connector_PinHeader_2.54mm:PinHeader_1x04_P2.54mm_Vertical, symbol Component_Library_Bavo:GY-NEO6MV2_Breakout
- added B5: GY-SGP41_Breakout, Connector_PinHeader_2.54mm:PinHeader_1x04_P2.54mm_Vertical, symbol Component_Library_Bavo:GY-SGP41_Breakout
- added B6: SCD41_Breakout, Connector_PinHeader_2.54mm:PinHeader_1x04_P2.54mm_Vertical, symbol Component_Library_Bavo:SCD41_Breakout
- added C4: 1µF, Capacitor_SMD:C_0805_2012Metric_Pad1.18x1.45mm_HandSolder, symbol Device:C_Small
- added C5: 100nF, Capacitor_SMD:C_0805_2012Metric_Pad1.18x1.45mm_HandSolder, symbol Device:C_Small
- added J4: SPS30_JST-ZHR-5, Connector_JST:JST_XH_B5B-XH-A_1x05_P2.50mm_Vertical, symbol Component_Library_Bavo:SPS30_JST-ZHR-5
- B1: value (none) -> DFROBOT-DFR0559; footprint (none) -> Component_Library_Bavo:DFROBOT-DFR0559
- B3: renamed from B2; value (none) -> CCS811_Breakout; footprint (none) -> Component_Library_Bavo:CCS811_Breakout
- B4: renamed from B3; value (none) -> BME280_Breakout; footprint (none) -> Component_Library_Bavo:BM280_Breakout
- B7: renamed from B4; value (none) -> DHT22_Breakout; footprint (none) -> Connector_PinHeader_2.54mm:PinHeader_1x04_P2.54mm_Vertical
- C1, C3: value (none) -> 1µF; footprint (none) -> Capacitor_SMD:C_0805_2012Metric_Pad1.18x1.45mm_HandSolder
- C10: renamed from C8; value (none) -> 100nF; footprint (none) -> Capacitor_SMD:C_0805_2012Metric_Pad1.18x1.45mm_HandSolder
- C2, C6: value (none) -> 100nF; footprint (none) -> Capacitor_SMD:C_0805_2012Metric_Pad1.18x1.45mm_HandSolder
- C7: renamed from C4; value (none) -> 100nF; footprint (none) -> Capacitor_SMD:C_0805_2012Metric_Pad1.18x1.45mm_HandSolder
- C8: renamed from C5; value (none) -> 100nF; footprint (none) -> Capacitor_SMD:C_0805_2012Metric_Pad1.18x1.45mm_HandSolder
- C9: renamed from C7; value (none) -> 100nF; footprint (none) -> Capacitor_SMD:C_0805_2012Metric_Pad1.18x1.45mm_HandSolder
- D1, D2, D3, D4, D5, D6, D7, D8, D9: value (none) -> LED; footprint (none) -> LED_SMD:LED_0805_2012Metric_Pad1.15x1.40mm_HandSolder
- H1, H2, H3, H4: value (none) -> MountingHole; footprint (none) -> MountingHole:MountingHole_3.2mm_M3_Pad_Via
- IC1: value (none) -> LDL1117S33R; footprint (none) -> Component_Library_Bavo:SOT95P280X145-5N
- J1: renamed from J2; value (none) -> Conn_01x03_Male; footprint (none) -> Connector_PinHeader_2.54mm:PinHeader_1x03_P2.54mm_Vertical
- J2: renamed from J3; value (none) -> SDS011_JST-XH-5; footprint (none) -> Connector_JST:JST_XH_B5B-XH-A_1x05_P2.50mm_Vertical
- J3: renamed from J4; value (none) -> Conn_01x03_Male; footprint (none) -> Connector_PinHeader_2.54mm:PinHeader_1x03_P2.54mm_Vertical
- J5: renamed from J6; value (none) -> Conn_01x03_Male; footprint (none) -> Connector_PinHeader_2.54mm:PinHeader_1x03_P2.54mm_Vertical
- R1, R10, R2, R3, R4, R5, R6, R7, R9: value (none) -> 1kΩ; footprint (none) -> Resistor_SMD:R_0805_2012Metric_Pad1.20x1.40mm_HandSolder
- R8: value (none) -> 10kΩ; footprint (none) -> Resistor_SMD:R_0805_2012Metric_Pad1.20x1.40mm_HandSolder
- U1: value (none) -> FLWSB-SAMDaaNo21-v1; footprint (none) -> Component_Library_Bavo:FLWSB-SAMDaaNo21-v1
Connections:
- net +3V3: now also B2.1 (VCC), B5.1 (VIN), B6.2 (VDD), C5.1
- net +5V: now also C4.1, J4.1 (VDD)
- net GND2: now also B2.4 (GND), B5.2 (GND), B6.1 (GND), C4.2, C5.2, J4.4 (SEL), J4.5 (GND)
- net S0RX-SDS: no longer J2.2 (RXD)
- net S0TX-SDS: no longer J2.1 (TXD), U1.6 (PA04)
- net SCL: now also B5.3 (SCL), B6.3 (SCL), J4.3 (TX/SCL)
- net SDA: now also B5.4 (SDA), B6.4 (SDA), J4.2 (RX/SDA)
- net S2RX-LoRa renamed S2TX-LoRa_RX
- net S2TX-LoRa_RX: now also U1.10 (PA08); no longer U1.11 (PA09)
- net S2TX-LoRa renamed S2RX-LoRa_TX
- net S2RX-LoRa_TX: now also U1.11 (PA09); no longer U1.10 (PA08)
- net S5RX renamed S5TX-EXTRA_RX
- net S5TX-EXTRA_RX: now also B2.2 (RX)
- net S5TX renamed S5RX-EXTRA_TX
- net S5RX-EXTRA_TX: now also B2.3 (TX)
- net SORX-SDS renamed S0RX-SDS_TX
- net S0RX-SDS_TX: now also J2.1 (TXD)
- new net SOTX-SDS_RX: J2.2 (RXD), U1.6 (PA04)
Other:
- note added: "Extra I2C connectors"
- note added: "SEL to GND to select I2C"
- note removed: "Extra I2C connector."
- moved on the sheet: B3, B4, C1, C2, C7, C8, D1, D2, D3, D4, D5, D6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
